Commit message: WIP add dynamic obstacles with controllers

File: resources/models/environment_assets/objects/cube.urdf (robot description, URDF)
Before this commit: robot box, 1 links, 0 joints
Links:
- link base_link: geometry 

File: resources/models/environment_assets/walls/back_wall.urdf (robot description, URDF)
Before this commit: robot back_wall, 1 links, 0 joints
Links:
- link base_link: geometry collision box size=0.2 20 10; visual box size=0.2 20 10

File: resources/models/environment_assets/walls/front_wall.urdf (robot description, URDF)
Before this commit: robot front_wall, 1 links, 0 joints
Links:
- link base_link: geometry collision box size=0.2 20 10; visual box size=0.2 20 10

File: resources/models/environment_assets/walls/left_wall.urdf (robot description, URDF)
Before this commit: robot left_wall, 1 links, 0 joints
Links:
- link base_link: geometry collision box size=20 0.2 10; visual box size=20 0.2 10

File: resources/models/environment_assets/walls/right_wall.urdf (robot description, URDF)
Before this commit: robot right_wall, 1 links, 0 joints
Links:
- link base_link: geometry collision box size=20 0.2 10; visual box size=20 0.2 10
