Commit message: Add pole like envs

File: resources/models/environment_assets/objects/cuboidal_rod.urdf (robot description, URDF)
Before this commit: robot box, 1 links, 0 joints
Links:
- link base_link: geometry collision box size=0.6 0.15 20.0; visual box size=0.6 0.15 20.0

Commit message: Thinner walls

File: resources/models/environment_assets/objects/cuboidal_rod.urdf (robot description, URDF)
Before this commit: robot box, 1 links, 0 joints
Links:
- link base_link: geometry collision box size=0.75 0.15 20.0; visual box size=0.75 0.15 20.0

Commit message: Draw trajectories at the end

File: resources/models/environment_assets/objects/cuboidal_rod.urdf (robot description, URDF)
Before this commit: robot box, 1 links, 0 joints
Links:
- link base_link: geometry collision box size=1.25 0.15 20.0; visual box size=1.25 0.15 20.0
