Commit message: Add skydio 2 mesh to the quad urdf

File: resources/robots/quad/model.urdf (robot description, URDF)
Before this commit: robot quadrotor, 5 links, 4 joints
Links:
- link back_left_prop: geometry 
- link back_right_prop: geometry 
- link base_link: geometry collision sphere radius=0.2; visual mesh filename=package://skydio_2_1000_poly.obj scale=0.002 0.002 0.002
- link front_left_prop: geometry 
- link front_right_prop: geometry 

Commit message: wip

File: resources/robots/quad/model.urdf (robot description, URDF)
Before this commit: robot quadrotor, 5 links, 4 joints
Links:
- link back_left_prop: geometry visual cylinder length=0.07 radius=0.05
- link back_right_prop: geometry visual cylinder length=0.07 radius=0.05
- link base_link: geometry collision sphere radius=0.2; visual cylinder length=0.025 radius=0.2
- link front_left_prop: geometry visual cylinder length=0.07 radius=0.05
- link front_right_prop: geometry visual cylinder length=0.07 radius=0.05

Commit message: quad urdf!

File: resources/robots/quad/model.urdf (robot description, URDF)
Before this commit: robot quadrotor, 5 links, 4 joints
Links:
- link base_link: geometry collision sphere radius=0.20; visual cylinder length=0.025 radius=0.2
